File: KiCad/VCU_Module/MCU.kicad_sch (KiCad schematic)
At the start: 21 parts, among them IC1 STM32C092RCT6, J11 Conn_ST_STDC14, SW2 SW_Push, U6 MCP2562FDT-H_SN

Commit message: added peripherals to mcu
Connections:
- net ADC0: now reaches IC1.17 (PA0)
- net ADC1: now reaches IC1.18 (PA1)
- net SPI1_NSS: now reaches IC1.21 (PA4)
- net SPI1_SCK: now reaches IC1.22 (PA5)
- net SPI1_MISO: now reaches IC1.23 (PA6)
- net SPI1_MOSI: now reaches IC1.24 (PA7)
- net TIM2_CH1: now reaches IC1.25 (PC4)
- net TIM2_CH2: now reaches IC1.26 (PC5)
- net TIM3_CH3: now reaches IC1.27 (PB0)
- net TIM3_CH4: now reaches IC1.28 (PB1)
- net I2C1_SCL: now reaches IC1.37 (PA9)
- net I2C1_SDA: now reaches IC1.42 (PA10)
- net PB3: now reaches IC1.57 (PB3)
- net PB3: now also J11.8 (JTDO/SWO)
- no-connect marks 51 -> 37
