File: KiCad/VCU_Module/MCU.kicad_sch (KiCad schematic)
At the start: 21 parts, among them IC1 STM32C092RCT6, J11 Conn_ST_STDC14, J8 Termination Resistor Jumper, SW2 SW_Push, U6 MCP2562FDT-H_SN

Commit message: finalized BOM
Parts:
- C13, C15, C16, C17: DIS (none) -> DigiKey; DPN (none) -> 490-5825-1-ND; MFR (none) -> Murata Electronics; MPN (none) -> GCJ21BR72A104KA01L; Purchase Link (none) -> https://www.digikey.com/en/products/detail/murata-electroni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
- C14: DIS (none) -> DigiKey; DPN (none) -> 445-6974-1-ND; MFR (none) -> TDK; MPN (none) -> CGA4J3X7S2A105K125AB; Purchase Link (none) -> https://www.digikey.com/en/products/detail/tdk/CGA4J3X7S2A1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
- D2: DPN 160-1179-1-ND -> 1516-QBLP631-2IBCT-ND; MFR Lite-On Inc. -> QT Brightek (QTB); MPN LTST-C170GKT -> QBLP631-2IB; Purchase Link https://www.digikey.com/en/products/detail/liteon/LTST-C170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 -> https://www.digikey.com/en/products/detail/qt-brightek-qtb/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
- J8: DIS (none) -> DigiKey; DPN (none) -> 612-TS-102-T-A-ND; MFR (none) -> Samtec Inc.; MPN (none) -> TS-102-T-A; Purchase Link (none) -> https://www.digikey.com/en/products/detail/samtec-inc/TS-10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
- R25: DPN 311-10.0KCRCT-ND -> 2019-SG73S2ATTD103JCT-ND; MFR YAGEO -> KOA Speer Electronics, Inc.; MPN RC0805FR-0710KL -> SG73S2ATTD103J; Purchase Link https://www.digikey.com/en/products/detail/yageo/RC0805FR-0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 -> https://www.digikey.com/en/products/detail/koa-speer-electr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
- R26: DPN 311-10.0KCRCT-ND -> 2019-SG73S2ATTD1200FCT-ND; MFR YAGEO -> KOA Speer Electronics, Inc.; MPN RC0805FR-0710KL -> SG73S2ATTD1200F; Purchase Link https://www.digikey.com/en/products/detail/yageo/RC0805FR-0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 -> https://www.digikey.com/en/products/detail/koa-speer-electr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
- R3: DPN 311-1.00KCRCT-ND -> 2019-SG73S2ATTD3600FCT-ND; MFR YAGEO -> KOA Speer Electronics, Inc.; MPN RC0805FR-071KL -> SG73S2ATTD3600F; Purchase Link https://www.digikey.com/en/products/detail/yageo/RC0805FR-0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 -> https://www.digikey.com/en/products/detail/koa-speer-electr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
- R9: DPN 311-1.00KCRCT-ND -> 2019-SG73S2ATTD6800FCT-ND; MFR YAGEO -> KOA Speer Electronics, Inc.; MPN RC0805FR-071KL -> SG73S2ATTD6800F; Purchase Link https://www.digikey.com/en/products/detail/yageo/RC0805FR-0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 -> https://www.digikey.com/en/products/detail/koa-speer-electr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

Commit message: final PCB fix
Parts:
- CR2: symbol ESDCAN03-2BWY:ESDCAN03-2BWY -> VMS_Symbols:ESDCAN03-2BWY
- CR3: footprint VMS_Footprints:ESDA051-1JY -> Diode_SMD:D_SOD-323; symbol ESDA051-1JY:ESDA051-1JY -> VMS_Symbols:ESDA051-1JY
- D5: value GRN -> Amber; DPN 160-1179-1-ND -> 732-150080AS75000CT-ND; MFR Lite-On Inc. -> Würth Elektronik; MPN LTST-C170GKT -> 150080AS75000; Purchase Link https://www.digikey.com/en/products/detail/liteon/LTST-C170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 -> https://www.digikey.com/en/products/detail/w%C3%BCrth-elekt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
- IC1: symbol STM32C092RCT6:STM32C092RCT6 -> VMS_Symbols:STM32C092RCT6
- R3: value 360 -> 1k; DPN 2019-SG73S2ATTD3600FCT-ND -> 2019-SG73S2ATTD1001FCT-ND; MPN SG73S2ATTD3600F -> SG73S2ATTD1001F; Purchase Link https://www.digikey.com/en/products/detail/koa-speer-electronics-inc/SG73S2ATTD3600F/10279941 -> https://www.digikey.com/en/products/detail/koa-speer-electronics-inc/SG73S2ATTD1001F/10279896
- R9: value 680 -> 1k; DPN 2019-SG73S2ATTD6800FCT-ND -> 2019-SG73S2ATTD1001FCT-ND; MPN SG73S2ATTD6800F -> SG73S2ATTD1001F; Purchase Link https://www.digikey.com/en/products/detail/koa-speer-electronics-inc/SG73S2ATTD6800F/10279885 -> https://www.digikey.com/en/products/detail/koa-speer-electronics-inc/SG73S2ATTD1001F/10279896
- U6: symbol MCP2562FDT-H_SN:MCP2562FDT-H_SN -> VMS_Symbols:MCP2562FDT-H_SN
Connections:
- net SWCLK/BOOT0: now also J11.4 (JTMS/SWDIO); no longer J11.6 (JCLK/SWCLK)
- net SWDIO: now also J11.6 (JCLK/SWCLK); no longer J11.4 (JTMS/SWDIO)
- net at R3.1: now also D5.2 (A); no longer D2.2 (A)
- net at R9.1: now also D2.2 (A); no longer D5.2 (A)
Other:
- note added: "Internal weak pull-up on NRST"

Commit message: updating components with AEC certified ones
Parts:
- C13, C14, C15, C16, C17, R25, R26, R3, R9: Automotive Certification (none) -> AEC-Q200
- CR2, CR3: Automotive Certification (none) -> AEC-Q101
- D2: Automotive Certification (none) -> AEC-Q102; DPN 1516-QBLP631-2IBCT-ND -> 846-1207-1-ND; MFR QT Brightek (QTB) -> Rohm Semiconductor; MPN QBLP631-2IB -> SMLMN2BCTT86C; Purchase Link https://www.digikey.com/en/products/detail/qt-brightek-qtb/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 -> https://www.digikey.com/en/products/detail/rohm-semiconduct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
- D5: Automotive Certification (none) -> AEC-Q101; DPN 732-150080AS75000CT-ND -> SML-H12D8TT86CCT-ND; MFR Würth Elektronik -> Rohm Semiconductor; MPN 150080AS75000 -> SML-H12D8TT86C; Purchase Link https://www.digikey.com/en/products/detail/w%C3%BCrth-elekt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 -> https://www.digikey.com/en/products/detail/rohm-semiconduct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
- IC1, J11, J8, SW2: Automotive Certification (none) -> None
- U6: Automotive Certification (none) -> AEC-Q100
