File: KiCad/VCU_Module/POWER.kicad_sch (KiCad schematic)
At the start: 18 parts, among them Q1 AO3401A, U1 OKI-78SR-5_1.5-W36-C, U2 TLV75533PDBV

Commit message: comments from andrew
Other:
- note added: "use a tps series switching power supply, at least 30V MHz class of switching frequencies, internal fets, sychronous rectification, do two of these, 1 for 5v and 1 for 3.3v, package with leads"
Changed lines of the file:
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@@
+		)
+	)
+	(text "use a tps series switching power supply, at least 30V MHz class of switching frequencies, internal fets, sychronous rectification, do two of these, 1 for 5v and 1 for 3.3v, package with leads"
+		(exclude_from_sim no)
+		(at 204.978 106.426 0)
+		(effects
+			(font
+				(size 1.27 1.27)
+				(thickness 0.254)
+				(bold yes)
+			)
 		)
 	)
