File: KiCad/VCU_Module/VCU_Module.kicad_pcb (KiCad board)
At the start: 2 copper layers, 85.2 x 107.8 mm, 66 parts, among them IC1 STM32C092RCT6, J1 5810132011, J10 12V, J11 Conn_ST_STDC14, J12 MCU1, J13 MCU2, J14 5V, J15 3V3, J16 MCU3, J17 MCU4, J2 CN1, J3 CN2, J4 CN3, J5 MCU6, J6 CN4, J7 MCU5, J8 Termination Resistor Jumper, J9 GND, Q1 SUD19P06-60, SW2 SW_Push, U3 LMR33640DDDA, U4 LMR33640DDDA, U6 MCP2562FDT-H_SN

Commit message: updating components with AEC certified ones
Parts:
- CR1: value MMSZ5245B-7-F -> SZMMSZ5245BT1G
- Q1: value SUD19P06-60 -> PJD9P06A-AU_L2_000A1
