File: KiCad/VCU_Module/VCU_Module.kicad_sch (KiCad schematic)
At the start: 47 parts, among them J1 5810132011, J10 12V, J12 MCU1, J13 MCU2, J14 5V, J15 3V3, J16 MCU3, J17 MCU4, J2 CN1, J3 CN2, J4 CN3, J5 MCU6, J6 CN4, J7 MCU5, J9 GND, Q1 PJD9P06A-AU_L2_000A1, U3 LMR33640DDDA, U4 LMR33640DDDA

Commit message: Successful run of build Makefile
Parts:
- F2: footprint (none) -> Fuse:Fuse_Blade_Mini_directSolder
- J12, J13, J16, J17, J2, J3: symbol Connector_Generic:Conn_01x10 -> VMS_Symbols:Conn_01x10
- N1: footprint N/A -> Package_SIP:SIP9_Housing; symbol Mechanical:Housing -> VMS_Symbols:Housing
Changed lines of the file:
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@@
 	)
 	(symbol
-		(lib_id "Connector_Generic:Conn_01x10")
+		(lib_id "VMS_Symbols:Conn_01x10")
 		(at 350.52 213.36 0)
 		(unit 1)
@@
 	)
 	(symbol
-		(lib_id "Connector_Generic:Conn_01x10")
+		(lib_id "VMS_Symbols:Conn_01x10")
 		(at 67.31 48.26 0)
 		(unit 1)
@@
 	)
 	(symbol
-		(lib_id "Connector_Generic:Conn_01x10")
+		(lib_id "VMS_Symbols:Conn_01x10")
 		(at 290.83 175.26 0)
 		(mirror y)
@@
 	)
 	(symbol
-		(lib_id "Connector_Generic:Conn_01x10")
+		(lib_id "VMS_Symbols:Conn_01x10")
 		(at 290.83 213.36 0)
 		(mirror y)
@@
 		(unit 1)
 		(body_style 1)
-		(exclude_from_sim yes)
+		(exclude_from_sim no)
 		(in_bom yes)
 		(on_board no)
-		(in_pos_files no)
+		(in_pos_files yes)
 		(dnp yes)
 		(property "Reference" "F2"
@@
 			)
 		)
-		(property "Footprint" ""
+		(property "Footprint" "Fuse:Fuse_Blade_Mini_directSolder"
 			(at 26.162 154.94 90)
 			(hide yes)
@@
 	)
 	(symbol
-		(lib_id "Mechanical:Housing")
+		(lib_id "VMS_Symbols:Housing")
 		(at 91.44 36.83 0)
 		(unit 1)
 		(body_style 1)
-		(exclude_from_sim yes)
+		(exclude_from_sim no)
 		(in_bom yes)
 		(on_board no)
-		(in_pos_files no)
+		(in_pos_files yes)
 		(dnp no)
 		(property "Reference" "N1"
@@
 			)
 		)
-		(property "Footprint" "N/A"
+		(property "Footprint" "Package_SIP:SIP9_Housing"
 			(at 92.71 35.56 0)
 			(hide yes)
@@
 			)
 		)
-		(property "Description" "Polymer, Glass Filled Enclosure 5.130\" L x 4.550\" W x 1.670\" H (130.30mm x 115.57mm x 42.42mm) Black"
+		(property "Description" "Housing"
 			(at 91.44 36.83 0)
 			(hide yes)
@@
 			)
 		)
-		(property "Datasheet" "https://www.onsemi.com/pdf/datasheet/mmsz5221bt1-d.pdf"
+		(property "Datasheet" "MMSZ5245B-7-F"
 			(at 63.5 184.15 0)
 			(hide yes)
@@
 	)
 	(symbol
-		(lib_id "Connector_Generic:Conn_01x10")
+		(lib_id "VMS_Symbols:Conn_01x10")
 		(at 26.67 48.26 0)
 		(mirror y)
@@
 	)
 	(symbol
-		(lib_id "Connector_Generic:Conn_01x10")
+		(lib_id "VMS_Symbols:Conn_01x10")
 		(at 290.83 148.59 0)
 		(mirror y)
