File: PCB/Wire_Harness/Motor Controller.kicad_sch (KiCad schematic)
At the start: 2 parts, among them J4 Motor Controller A, J6 Motor Controller B

Commit message: Adding molex connectors for main bus and modules
Other:
- company: (none) -> Viking Motorsports
- title: (none) -> Formula EV Wiring Diagram
Changed lines of the file:
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@@
 	(generator_version "10.0")
 	(paper "A4")
+	(title_block
+		(title "Formula EV Wiring Diagram")
+		(date "2026-08-17")
+		(rev "1.0")
+		(company "Viking Motorsports")
+	)
 	(hierarchical_label "GPIO4"
 		(shape bidirectional)
