File: PCB/VCU_Module/MCU.kicad_sch (KiCad schematic)
At the start: 21 parts, among them IC1 STM32C092RCT6, J11 Conn_ST_STDC14, J8 Termination Resistor Jumper, SW2 SW_Push, U6 MCP2562FDT-H_SN

Commit message: move STLink connector and change component to correct version with alignment tabs
Parts:
- J11: DPN 612-FTSH-107-01-F-DV-K-ND -> SAM12420-ND; MPN FTSH-107-01-F-DV-K -> FTSH-107-01-S-D-K; Purchase Link https://www.digikey.com/en/products/detail/samtec-inc/FTSH-107-01-F-DV-K/2650001 -> https://www.digikey.com/en/products/detail/samtec-inc/FTSH-107-01-S-D-K/2650004?gclsrc=aw.ds&gad_source=1&gad_campaignid=17336967819&gbraid=0AAAAADrbLlicyKK0eY_V0wleFKoDjVbWz&gclid=CjwKCAjw1vXTBhB-EiwAEKr_k6pgiYkH2W21gU4f999biLNDO9FzNBRms_SrUikYiU-KfRn2oXJkshoCrk8QAvD_BwE
Changed lines of the file:
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@@
 			)
 		)
-		(property "Datasheet" "https://www.st.com/content/ccc/resource/technical/document/user_manual/group1/99/49/91/b6/b2/3a/46/e5/DM00526767/files/DM00526767.pdf/jcr:content/translations/en.DM00526767.pdf"
+		(property "Datasheet" "https://suddendocs.samtec.com/catalog_english/ftsh_th.pdf"
 			(at 31.75 143.51 90)
 			(hide yes)
@@
 			)
 		)
-		(property "DPN" "612-FTSH-107-01-F-DV-K-ND"
+		(property "DPN" "SAM12420-ND"
 			(at 40.64 111.76 0)
 			(hide yes)
@@
 			)
 		)
-		(property "MPN" "FTSH-107-01-F-DV-K"
+		(property "MPN" "FTSH-107-01-S-D-K"
 			(at 40.64 111.76 0)
 			(hide yes)
@@
 			)
 		)
-		(property "Purchase Link" "https://www.digikey.com/en/products/detail/samtec-inc/FTSH-107-01-F-DV-K/2650001"
+		(property "Purchase Link" "https://www.digikey.com/en/products/detail/samtec-inc/FTSH-107-01-S-D-K/2650004?gclsrc=aw.ds&gad_source=1&gad_campaignid=17336967819&gbraid=0AAAAADrbLlicyKK0eY_V0wleFKoDjVbWz&gclid=CjwKCAjw1vXTBhB-EiwAEKr_k6pgiYkH2W21gU4f999biLNDO9FzNBRms_SrUikYiU-KfRn2oXJkshoCrk8QAvD_BwE"
 			(at 40.64 111.76 0)
 			(hide yes)

Commit message: fixing header labeling issue, replacing headers with lower profile versions
Parts:
- J8: Purchase Link https://www.digikey.com/en/products/detail/samtec-inc/TS-10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 -> https://www.digikey.com/en/products/detail/preci-dip/310-87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
Changed lines of the file:
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@@
 			)
 		)
-		(property "Datasheet" "https://suddendocs.samtec.com/catalog_english/td.pdf"
+		(property "Datasheet" "https://mm.digikey.com/Volume0/opasdata/d220001/medias/docus/8890/PdfFile_256753.pdf"
 			(at 115.57 227.33 0)
 			(hide yes)
@@
 			)
 		)
-		(property "Purchase Link" "https://www.digikey.com/en/products/detail/samtec-inc/TS-102-T-A/1105492"
+		(property "Purchase Link" "https://www.digikey.com/en/products/detail/preci-dip/310-87-104-41-001101/3757342"
 			(at 115.57 227.33 0)
 			(hide yes)

Commit message: Ran makefile successfully
Parts:
- renumbered C14 to C15, C15 to C16, C13 to C17, C16 to C18, C17 to C19, CR3 to CR2, CR2 to CR3, D5 to D3, D2 to D4, J11 to J16, J8 to J17, R25 to R10, R26 to R11, R3 to R8, SW2 to SW1, TP12 to TP1, TP13 to TP2, TP14 to TP3, U6 to U3
