File: PCB/VCU_Module/VCU_Module.kicad_pcb (KiCad board)
At the start: 2 copper layers, 85.2 x 107.8 mm, 66 parts, among them IC1 STM32C092RCT6, J1 5810132011, J10 12V, J11 Conn_ST_STDC14, J12 MCU1, J13 MCU2, J14 5V, J15 3V3, J16 MCU3, J17 MCU4, J2 CN1, J3 CN2, J4 CN3, J5 MCU6, J6 CN4, J7 MCU5, J8 Termination Resistor Jumper, J9 GND, Q1 PJD9P06A-AU_L2_000A1, SW2 SW_Push, U3 LMR33640DDDA, U4 LMR33640DDDA, U6 MCP2562FDT-H_SN

Commit message: fixing header labeling issue, replacing headers with lower profile versions
Parts:
- J10: value 12V -> 310-83-102-41-001101-ND
- J12: value MCU1 -> 801-87-010-10-012101
- J13: value MCU2 -> 801-87-010-10-012101
- J14: value 5V -> 310-87-104-41-001101
- J15: value 3V3 -> 310-87-104-41-001101
- J16: value MCU3 -> 801-87-010-10-012101
- J17: value MCU4 -> 801-87-010-10-012101
- J2: value CN1 -> 801-87-010-10-012101
- J3: value CN2 -> 801-87-010-10-012101
- J4: value CN3 -> 801-87-006-10-012101
- J5: value MCU6 -> 310-87-104-41-001101
- J6: value CN4 -> 801-87-006-10-012101
- J7: value MCU5 -> 801-87-006-10-012101
- J9: value GND -> 310-87-104-41-001101
Other:
- board text added: "12V"
- board text added: "3V"
- board text added: "5V"

Commit message: Ran makefile successfully
Parts:
- renumbered C5 to C1, C11 to C10, C19 to C11, C20 to C12, C21 to C13, C12 to C14, C14 to C15, C15 to C16, C13 to C17, C16 to C18, C17 to C19, C3 to C2, C4 to C3, C6 to C4, C7 to C5, C8 to C6, C9 to C7, C18 to C8, C10 to C9, CR3 to CR2, CR2 to CR3, D4 to D2, D5 to D3, D2 to D4, J2 to J1, J16 to J10, J17 to J11, J14 to J12, J10 to J13, J9 to J14, J11 to J16, J8 to J17, J1 to J2, J6 to J5, J12 to J6, J5 to J7, J13 to J8, J7 to J9, R4 to R1, R25 to R10, R26 to R11, R5 to R3, R1 to R4, R6 to R5, R8 to R6, R3 to R8, SW2 to SW1, TP12 to TP1, TP13 to TP2, TP14 to TP3, U3 to U1, U4 to U2, U6 to U3
