File: PCB/VCU_Module/VCU_Module.kicad_sch (KiCad schematic)
At the start: 47 parts, among them J1 5810132011, J10 12V, J12 MCU1, J13 MCU2, J14 5V, J15 3V3, J16 MCU3, J17 MCU4, J2 CN1, J3 CN2, J4 CN3, J5 MCU6, J6 CN4, J7 MCU5, J9 GND, Q1 PJD9P06A-AU_L2_000A1, U3 LMR33640DDDA, U4 LMR33640DDDA

Commit message: fixing header labeling issue, replacing headers with lower profile versions
Parts:
- J10: value 12V -> 310-83-102-41-001101-ND; DPN S7035-ND -> 310-83-102-41-001101-ND; MFR Sullins Connector Solutions -> Preci-Dip; MPN PPPC021LFBN-RC -> 310-83-102-41-001101; Purchase Link https://www.digikey.com/en/products/detail/sullins-connecto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 -> https://www.digikey.com/en/products/detail/preci-dip/310-83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
- J12: value MCU1 -> 801-87-010-10-012101; DPN S7043-ND -> 1212-1197-ND; MFR Sullins Connector Solutions -> Preci-Dip; MPN PPPC101LFBN-RC -> 801-87-010-10-012101; Purchase Link https://www.digikey.com/en/products/detail/sullins-connecto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 -> https://www.digikey.com/en/products/detail/preci-dip/801-87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
- J13: value MCU2 -> 801-87-010-10-012101; DPN S7043-ND -> 1212-1197-ND; MFR Sullins Connector Solutions -> Preci-Dip; MPN PPPC101LFBN-RC -> 801-87-010-10-012101; Purchase Link https://www.digikey.com/en/products/detail/sullins-connecto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 -> https://www.digikey.com/en/products/detail/preci-dip/801-87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
- J14: value 5V -> 310-87-104-41-001101; DPN S7037-ND -> 1212-1092-ND; MFR Sullins Connector Solutions -> Preci-Dip; MPN PPPC041LFBN-RC -> 310-87-104-41-001101
- J15: value 3V3 -> 310-87-104-41-001101; DPN S7037-ND -> 1212-1092-ND; MFR Sullins Connector Solutions -> Preci-Dip; MPN PPPC041LFBN-RC -> 310-87-104-41-001101
- J16: value MCU3 -> 801-87-010-10-012101; DPN S7043-ND -> 1212-1197-ND; MFR Sullins Connector Solutions -> Preci-Dip; MPN PPPC101LFBN-RC -> 801-87-010-10-012101; Purchase Link https://www.digikey.com/en/products/detail/sullins-connecto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 -> https://www.digikey.com/en/products/detail/preci-dip/801-87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
- J17: value MCU4 -> 801-87-010-10-012101; DPN S7043-ND -> 1212-1197-ND; MFR Sullins Connector Solutions -> Preci-Dip; MPN PPPC101LFBN-RC -> 801-87-010-10-012101; Purchase Link https://www.digikey.com/en/products/detail/sullins-connecto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 -> https://www.digikey.com/en/products/detail/preci-dip/801-87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
- J2: value CN1 -> 801-87-010-10-012101; DPN S7043-ND -> 1212-1197-ND; MFR Sullins Connector Solutions -> Preci-Dip; MPN PPPC101LFBN-RC -> 801-87-010-10-012101; Purchase Link https://www.digikey.com/en/products/detail/sullins-connecto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 -> https://www.digikey.com/en/products/detail/preci-dip/801-87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
- J3: value CN2 -> 801-87-010-10-012101; DPN S7043-ND -> 1212-1197-ND; MFR Sullins Connector Solutions -> Preci-Dip; MPN PPPC101LFBN-RC -> 801-87-010-10-012101; Purchase Link https://www.digikey.com/en/products/detail/sullins-connecto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 -> https://www.digikey.com/en/products/detail/preci-dip/801-87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
- J4: value CN3 -> 801-87-006-10-012101; DPN S7039-ND -> 801-87-006-10-012101-ND; MFR Sullins Connector Solutions -> Preci-Dip; MPN PPPC061LFBN-RC -> 801-87-006-10-012101; Purchase Link https://www.digikey.com/en/products/detail/sullins-connecto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 -> https://www.digikey.com/en/products/detail/preci-dip/801-87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
- J5: value MCU6 -> 310-87-104-41-001101; DPN S7037-ND -> 1212-1092-ND; MFR Sullins Connector Solutions -> Preci-Dip; MPN PPPC041LFBN-RC -> 310-87-104-41-001101
- J6: value CN4 -> 801-87-006-10-012101; DPN S7039-ND -> 801-87-006-10-012101-ND; MFR Sullins Connector Solutions -> Preci-Dip; MPN PPPC061LFBN-RC -> 801-87-006-10-012101; Purchase Link https://www.digikey.com/en/products/detail/sullins-connecto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 -> https://www.digikey.com/en/products/detail/preci-dip/801-87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
- J7: value MCU5 -> 801-87-006-10-012101; DPN S7039-ND -> 801-87-006-10-012101-ND; MFR Sullins Connector Solutions -> Preci-Dip; MPN PPPC061LFBN-RC -> 801-87-006-10-012101; Purchase Link https://www.digikey.com/en/products/detail/sullins-connecto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 -> https://www.digikey.com/en/products/detail/preci-dip/801-87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
- J9: value GND -> 310-87-104-41-001101; DPN S7037-ND -> 1212-1092-ND; MFR Sullins Connector Solutions -> Preci-Dip; MPN PPPC041LFBN-RC -> 310-87-104-41-001101

Commit message: Ran makefile successfully
Parts:
- renumbered C5 to C1, C11 to C10, C19 to C11, C20 to C12, C21 to C13, C12 to C14, C3 to C2, C4 to C3, C6 to C4, C7 to C5, C8 to C6, C9 to C7, C18 to C8, C10 to C9, D4 to D2, J2 to J1, J16 to J10, J17 to J11, J14 to J12, J10 to J13, J9 to J14, J1 to J2, J6 to J5, J12 to J6, J5 to J7, J13 to J8, J7 to J9, R4 to R1, R5 to R3, R1 to R4, R6 to R5, R8 to R6, U3 to U1, U4 to U2
